Commit message: Added back left wheel and transmission

File: moon_description/robot/robot.urdf.xacro (robot description, xacro)
@@ -11,4 +11,7 @@
   <xacro:property name="base_height" value="0.06"/>
   <xacro:property name="caster_radius" value="0.03"/>
+  <xacro:property name="wheel_width" value="0.02"/>
+  <xacro:property name="wheel_radius" value="0.035"/>
+  <xacro:property name="wheel_holder_size" value="0.01"/>
  <link name="base_footprint">
     <visual>
@@ -45,5 +48,5 @@
     <parent link="base_link"/>
     <child link="caster_front_left_wheel"/>
-    <origin rpy="${-pi/2} 0 0" xyz="0.05 -0.1 0.006"/>
+    <origin rpy="${-pi/2} 0 0" xyz="0.05 -0.1 0"/>
   </joint>
  <link name="caster_front_right_wheel">
@@ -58,5 +61,47 @@
     <parent link="base_link"/>
     <child link="caster_front_right_wheel"/>
-    <origin rpy="${-pi/2} 0 0" xyz="-0.05 -0.1 0.006"/>
+    <origin rpy="${-pi/2} 0 0" xyz="-0.05 -0.1 0"/>
   </joint>
+  <link name="back_left_wheel_holder">
+    <visual>
+      <xacro:box_geometry width="${wheel_holder_size}" height="${wheel_holder_size}" depth="${wheel_holder_size}"/>
+      <xacro:green_material/>
+    </visual>
+    <xacro:box_collision width="${wheel_holder_size}" height="${wheel_holder_size}" depth="${wheel_holder_size}"/>
+    <xacro:box_inertia mass="0.003" width="${wheel_holder_size}" height="${wheel_holder_size}"
+                       depth="${wheel_holder_size}"/>
+  </link>
+  <joint name="base_to_back_left_wheel_holder" type="fixed">
+    <parent link="base_link"/>
+    <child link="back_left_wheel_holder"/>
+    <origin xyz="${wheel_holder_size/2 + 0.025} 0 ${wheel_holder_size/2}" rpy="0 0 0" />
+    <axis xyz="0 0 1" />
+  </joint>
+  <link name="back_left_wheel">
+    <visual>
+      <xacro:cylinder_geometry radius="${wheel_radius}" height="${wheel_width}"/>
+      <xacro:black_material/>
+    </visual>
+    <xacro:cylinder_collision radius="${wheel_radius}" height="${wheel_width}"/>
+    <xacro:cylinder_inertia mass="0.03" radius="${wheel_radius}" height="${wheel_width}"/>
+    <dynamics damping="0.01" friction="100.0" />
+  </link>
+  <joint name="back_left_wheel_joint" type="continuous">
+    <parent link="back_left_wheel_holder"/>
+    <child link="back_left_wheel"/>
+    <origin xyz="${wheel_width/2 + wheel_holder_size/2} 0 0" rpy="0 ${pi/2} 0" />
+    <axis xyz="0 0 1" />
+    <limit effort="100" velocity="100" />
+    <dynamics damping="0.01" friction="0.0" />
+  </joint>
+  <transmission name="back_left_wheel_transmission">
+     <type>transmission_interface/SimpleTransmission</type>
+     <joint name="back_left_wheel_joint">
+       <hardwareInterface>EffortJointInterface</hardwareInterface>
+     </joint>
+     <actuator name="back_left_wheel_motor">
+       <hardwareInterface>EffortJointInterface</hardwareInterface>
+       <mechanicalReduction>1</mechanicalReduction>
+     </actuator>
+  </transmission>
 </robot>

Commit message: Added macros for the wheels

File: moon_description/robot/robot.urdf.xacro (robot description, xacro)
@@ -1,107 +1,46 @@
 <?xml version="1.0"?>
 <robot name="moon" xmlns:xacro="http://ros.org/wiki/xacro">
-  <!-- Global constants -->
-  <xacro:property name="pi" value="3.1415926535897931"/>
-  <!-- Included files -->
-  <xacro:include filename="$(find moon_description)/urdf/materials.urdf.xacro"/>
-  <xacro:include filename="$(find moon_description)/urdf/common.urdf.xacro"/>
-   <!-- Robot properties -->
-  <xacro:property name="base_width" value="0.2"/>
-  <xacro:property name="base_length" value="0.26"/>
-  <xacro:property name="base_height" value="0.06"/>
-  <xacro:property name="caster_radius" value="0.03"/>
-  <xacro:property name="wheel_width" value="0.02"/>
-  <xacro:property name="wheel_radius" value="0.035"/>
-  <xacro:property name="wheel_holder_size" value="0.01"/>
- <link name="base_footprint">
-    <visual>
-      <xacro:box_geometry width="0.001" depth="0.001" height="0.001"/>
-      <xacro:white_material/>
-    </visual>
-    <xacro:box_inertia mass="0.0001" width="0.001" depth="0.001" height="0.001"/>
- </link>
-  <joint name="base_footprint_joint" type="fixed">
-    <origin rpy="0 0 0" xyz="0 0 0.04"/>
-    <parent link="base_footprint"/>
-    <child link="base_link"/>
-  </joint>
-  <link name="base_link">
-    <visual>
-        <origin xyz="0 0 0" rpy="0 0 0"/>
-        <geometry>
-            <mesh filename="package://moon_description/meshes/moon_base.stl"/>
-        </geometry>
-      <xacro:white_material/>
-    </visual>
-    <xacro:box_collision width="${base_width}" depth="${base_height}" height="${base_length}"/>
-    <xacro:box_inertia mass="3" width="${base_width}" depth="${base_height}" height="${base_length}"/>
-  </link>
- <link name="caster_front_left_wheel">
-    <visual>
-      <xacro:sphere_geometry radius="${caster_radius}"/>
-      <xacro:black_material/>
-    </visual>
-    <xacro:sphere_collision radius="${caster_radius}"/>
-    <xacro:sphere_inertia mass="0.05" radius="${caster_radius}"/>
-  </link>
-  <joint name="caster_front_left_joint" type="fixed">
-    <parent link="base_link"/>
-    <child link="caster_front_left_wheel"/>
-    <origin rpy="${-pi/2} 0 0" xyz="0.05 -0.1 0"/>
-  </joint>
- <link name="caster_front_right_wheel">
-    <visual>
-      <xacro:sphere_geometry radius="${caster_radius}"/>
-      <xacro:black_material/>
-    </visual>
-    <xacro:sphere_collision radius="${caster_radius}"/>
-    <xacro:sphere_inertia mass="0.05" radius="${caster_radius}"/>
-  </link>
-  <joint name="caster_front_right_joint" type="fixed">
-    <parent link="base_link"/>
-    <child link="caster_front_right_wheel"/>
-    <origin rpy="${-pi/2} 0 0" xyz="-0.05 -0.1 0"/>
-  </joint>
-  <link name="back_left_wheel_holder">
-    <visual>
-      <xacro:box_geometry width="${wheel_holder_size}" height="${wheel_holder_size}" depth="${wheel_holder_size}"/>
-      <xacro:green_material/>
-    </visual>
-    <xacro:box_collision width="${wheel_holder_size}" height="${wheel_holder_size}" depth="${wheel_holder_size}"/>
-    <xacro:box_inertia mass="0.003" width="${wheel_holder_size}" height="${wheel_holder_size}"
-                       depth="${wheel_holder_size}"/>
-  </link>
-  <joint name="base_to_back_left_wheel_holder" type="fixed">
-    <parent link="base_link"/>
-    <child link="back_left_wheel_holder"/>
-    <origin xyz="${wheel_holder_size/2 + 0.025} 0 ${wheel_holder_size/2}" rpy="0 0 0" />
-    <axis xyz="0 0 1" />
-  </joint>
-  <link name="back_left_wheel">
-    <visual>
-      <xacro:cylinder_geometry radius="${wheel_radius}" height="${wheel_width}"/>
-      <xacro:black_material/>
-    </visual>
-    <xacro:cylinder_collision radius="${wheel_radius}" height="${wheel_width}"/>
-    <xacro:cylinder_inertia mass="0.03" radius="${wheel_radius}" height="${wheel_width}"/>
-    <dynamics damping="0.01" friction="100.0" />
-  </link>
-  <joint name="back_left_wheel_joint" type="continuous">
-    <parent link="back_left_wheel_holder"/>
-    <child link="back_left_wheel"/>
-    <origin xyz="${wheel_width/2 + wheel_holder_size/2} 0 0" rpy="0 ${pi/2} 0" />
-    <axis xyz="0 0 1" />
-    <limit effort="100" velocity="100" />
-    <dynamics damping="0.01" friction="0.0" />
-  </joint>
-  <transmission name="back_left_wheel_transmission">
-     <type>transmission_interface/SimpleTransmission</type>
-     <joint name="back_left_wheel_joint">
-       <hardwareInterface>EffortJointInterface</hardwareInterface>
-     </joint>
-     <actuator name="back_left_wheel_motor">
-       <hardwareInterface>EffortJointInterface</hardwareInterface>
-       <mechanicalReduction>1</mechanicalReduction>
-     </actuator>
-  </transmission>
+    <!-- Global constants -->
+    <xacro:property name="pi" value="3.1415926535897931"/>
+    <!-- Included files -->
+    <xacro:include filename="$(find moon_description)/urdf/materials.urdf.xacro"/>
+    <xacro:include filename="$(find moon_description)/urdf/common.urdf.xacro"/>
+    <xacro:include filename="$(find moon_description)/urdf/wheels.urdf.xacro"/>
+    <!-- Robot properties -->
+    <xacro:property name="base_width" value="0.2"/>
+    <xacro:property name="base_length" value="0.26"/>
+    <xacro:property name="base_height" value="0.06"/>
+    <xacro:property name="caster_radius" value="0.03"/>
+    <xacro:property name="wheel_width" value="0.02"/>
+    <xacro:property name="wheel_radius" value="0.035"/>
+    <xacro:property name="wheel_holder_size" value="0.01"/>
+    <link name="base_footprint">
+        <visual>
+            <xacro:box_geometry width="0.001" depth="0.001" height="0.001"/>
+            <xacro:white_material/>
+        </visual>
+        <xacro:box_inertia mass="0.0001" width="0.001" depth="0.001" height="0.001"/>
+    </link>
+    <joint name="base_footprint_joint" type="fixed">
+        <origin rpy="0 0 0" xyz="0 0 0.03"/>
+        <parent link="base_footprint"/>
+        <child link="base_link"/>
+    </joint>
+    <link name="base_link">
+        <visual>
+            <origin xyz="0 0 0" rpy="0 0 0"/>
+            <geometry>
+                <mesh filename="package://moon_description/meshes/moon_base.stl"/>
+            </geometry>
+            <xacro:white_material/>
+        </visual>
+        <xacro:box_collision width="${base_width}" depth="${base_height}" height="${base_length}"/>
+        <xacro:box_inertia mass="3" width="${base_width}" depth="${base_height}" height="${base_length}"/>
+    </link>
+    <xacro:caster_wheel prefix="front_left" radius="${caster_radius}" x="0.05" y="-0.1" z="0"/>
+    <xacro:caster_wheel prefix="front_right" radius="${caster_radius}" x="-0.05" y="-0.1" z="0"/>
+    <xacro:transmission_wheel prefix="back_left" radius="${wheel_radius}" width="${wheel_width}"
+                              holder_size="${wheel_holder_size}" wheels_distance="0.05" direction="1.0"/>
+    <xacro:transmission_wheel prefix="back_right" radius="${wheel_radius}" width="${wheel_width}"
+                              holder_size="${wheel_holder_size}" wheels_distance="0.05" direction="-1.0"/>
 </robot>

Commit message: Added LIDAR link to URDF

File: moon_description/robot/robot.urdf.xacro (robot description, xacro)
@@ -15,4 +15,6 @@
     <xacro:property name="wheel_radius" value="0.035"/>
     <xacro:property name="wheel_holder_size" value="0.01"/>
+    <xacro:property name="lidar_height" value="0.02"/>
+    <xacro:property name="lidar_radius" value="0.04"/>
     <link name="base_footprint">
         <visual>
@@ -44,3 +46,17 @@
     <xacro:transmission_wheel prefix="back_right" radius="${wheel_radius}" width="${wheel_width}"
                               holder_size="${wheel_holder_size}" wheels_distance="0.05" direction="-1.0"/>
+    <link name="lidar">
+        <visual>
+            <xacro:cylinder_geometry radius="${lidar_radius}" height="${lidar_height}"/>
+            <xacro:green_material/>
+        </visual>
+        <xacro:cylinder_collision radius="${lidar_radius}" height="${lidar_height}"/>
+        <xacro:cylinder_inertia mass="0.1" radius="${lidar_radius}" height="${lidar_height}"/>
+        <dynamics damping="0.01" friction="100.0" />
+    </link>
+    <joint name="lidar_joint" type="fixed">
+        <origin rpy="0 0 0" xyz="0 0.04 ${base_height + lidar_height/2}"/>
+        <parent link="base_link"/>
+        <child link="lidar"/>
+    </joint>
 </robot>
