Commit message: Fixed indentation. Reduced configuration files and added Gazebo package first version.

File: moon_description/robot/robot.urdf.xacro (robot description, xacro)
@@ -1,62 +1,62 @@
 <?xml version="1.0"?>
 <robot name="moon" xmlns:xacro="http://ros.org/wiki/xacro">
-    <!-- Global constants -->
-    <xacro:property name="pi" value="3.1415926535897931"/>
-    <!-- Included files -->
-    <xacro:include filename="$(find moon_description)/urdf/materials.urdf.xacro"/>
-    <xacro:include filename="$(find moon_description)/urdf/common.urdf.xacro"/>
-    <xacro:include filename="$(find moon_description)/urdf/wheels.urdf.xacro"/>
-    <!-- Robot properties -->
-    <xacro:property name="base_width" value="0.2"/>
-    <xacro:property name="base_length" value="0.26"/>
-    <xacro:property name="base_height" value="0.06"/>
-    <xacro:property name="caster_radius" value="0.03"/>
-    <xacro:property name="wheel_width" value="0.02"/>
-    <xacro:property name="wheel_radius" value="0.035"/>
-    <xacro:property name="wheel_holder_size" value="0.01"/>
-    <xacro:property name="lidar_height" value="0.02"/>
-    <xacro:property name="lidar_radius" value="0.04"/>
-    <link name="base_footprint">
-        <visual>
-            <xacro:box_geometry width="0.001" depth="0.001" height="0.001"/>
-            <xacro:white_material/>
-        </visual>
-        <xacro:box_inertia mass="0.0001" width="0.001" depth="0.001" height="0.001"/>
-    </link>
-    <joint name="base_footprint_joint" type="fixed">
-        <origin rpy="0 0 0" xyz="0 0 0.03"/>
-        <parent link="base_footprint"/>
-        <child link="base_link"/>
-    </joint>
-    <link name="base_link">
-        <visual>
-            <origin xyz="0 0 0" rpy="0 0 0"/>
-            <geometry>
-                <mesh filename="package://moon_description/meshes/moon_base.stl"/>
-            </geometry>
-            <xacro:white_material/>
-        </visual>
-        <xacro:box_collision width="${base_width}" depth="${base_height}" height="${base_length}"/>
-        <xacro:box_inertia mass="3" width="${base_width}" depth="${base_height}" height="${base_length}"/>
-    </link>
-    <xacro:caster_wheel prefix="front_left" radius="${caster_radius}" x="0.05" y="-0.1" z="0"/>
-    <xacro:caster_wheel prefix="front_right" radius="${caster_radius}" x="-0.05" y="-0.1" z="0"/>
-    <xacro:transmission_wheel prefix="back_left" radius="${wheel_radius}" width="${wheel_width}"
-                              holder_size="${wheel_holder_size}" wheels_distance="0.05" direction="1.0"/>
-    <xacro:transmission_wheel prefix="back_right" radius="${wheel_radius}" width="${wheel_width}"
-                              holder_size="${wheel_holder_size}" wheels_distance="0.05" direction="-1.0"/>
-    <link name="lidar">
-        <visual>
-            <xacro:cylinder_geometry radius="${lidar_radius}" height="${lidar_height}"/>
-            <xacro:green_material/>
-        </visual>
-        <xacro:cylinder_collision radius="${lidar_radius}" height="${lidar_height}"/>
-        <xacro:cylinder_inertia mass="0.1" radius="${lidar_radius}" height="${lidar_height}"/>
-        <dynamics damping="0.01" friction="100.0" />
-    </link>
-    <joint name="lidar_joint" type="fixed">
-        <origin rpy="0 0 0" xyz="0 0.04 ${base_height + lidar_height/2}"/>
-        <parent link="base_link"/>
-        <child link="lidar"/>
-    </joint>
+  <!-- Global constants -->
+  <xacro:property name="pi" value="3.1415926535897931"/>
+  <!-- Included files -->
+  <xacro:include filename="$(find moon_description)/urdf/materials.urdf.xacro"/>
+  <xacro:include filename="$(find moon_description)/urdf/common.urdf.xacro"/>
+  <xacro:include filename="$(find moon_description)/urdf/wheels.urdf.xacro"/>
+  <!-- Robot properties -->
+  <xacro:property name="base_width" value="0.2"/>
+  <xacro:property name="base_length" value="0.26"/>
+  <xacro:property name="base_height" value="0.06"/>
+  <xacro:property name="caster_radius" value="0.03"/>
+  <xacro:property name="wheel_width" value="0.02"/>
+  <xacro:property name="wheel_radius" value="0.035"/>
+  <xacro:property name="wheel_holder_size" value="0.01"/>
+  <xacro:property name="lidar_height" value="0.02"/>
+  <xacro:property name="lidar_radius" value="0.04"/>
+  <link name="base_footprint">
+    <visual>
+      <xacro:box_geometry width="0.001" depth="0.001" height="0.001"/>
+      <xacro:white_material/>
+    </visual>
+    <xacro:box_inertia mass="0.0001" width="0.001" depth="0.001" height="0.001"/>
+  </link>
+  <joint name="base_footprint_joint" type="fixed">
+    <origin rpy="0 0 0" xyz="0 0 0.03"/>
+    <parent link="base_footprint"/>
+    <child link="base_link"/>
+  </joint>
+  <link name="base_link">
+    <visual>
+      <origin xyz="0 0 0" rpy="0 0 0"/>
+      <geometry>
+        <mesh filename="package://moon_description/meshes/moon_base.stl"/>
+      </geometry>
+      <xacro:white_material/>
+    </visual>
+    <xacro:box_collision width="${base_width}" depth="${base_height}" height="${base_length}"/>
+    <xacro:box_inertia mass="3" width="${base_width}" depth="${base_height}" height="${base_length}"/>
+  </link>
+  <xacro:caster_wheel prefix="front_left" radius="${caster_radius}" x="0.05" y="-0.1" z="0"/>
+  <xacro:caster_wheel prefix="front_right" radius="${caster_radius}" x="-0.05" y="-0.1" z="0"/>
+  <xacro:transmission_wheel prefix="back_left" radius="${wheel_radius}" width="${wheel_width}"
+                            holder_size="${wheel_holder_size}" wheels_distance="0.05" direction="1.0"/>
+  <xacro:transmission_wheel prefix="back_right" radius="${wheel_radius}" width="${wheel_width}"
+                            holder_size="${wheel_holder_size}" wheels_distance="0.05" direction="-1.0"/>
+  <link name="lidar">
+    <visual>
+      <xacro:cylinder_geometry radius="${lidar_radius}" height="${lidar_height}"/>
+      <xacro:green_material/>
+    </visual>
+    <xacro:cylinder_collision radius="${lidar_radius}" height="${lidar_height}"/>
+    <xacro:cylinder_inertia mass="0.1" radius="${lidar_radius}" height="${lidar_height}"/>
+    <dynamics damping="0.01" friction="100.0"/>
+  </link>
+  <joint name="lidar_joint" type="fixed">
+    <origin rpy="0 0 0" xyz="0 0.04 ${base_height + lidar_height/2}"/>
+    <parent link="base_link"/>
+    <child link="lidar"/>
+  </joint>
 </robot>

File: moon_description/urdf/common.urdf.xacro (robot description, xacro)
@@ -2,11 +2,11 @@
 <robot xmlns:xacro="http://www.ros.org/wiki/xacro">
   <xacro:macro name="sphere_inertia" params="mass radius">
-      <inertial>
-         <mass value="${mass}" />
-         <origin xyz="0 0 0" />
-         <inertia  ixx="${2*mass*radius*radius/5}" ixy="0.0" ixz="0.0"
-                   iyy="${2*mass*radius*radius/5}" iyz="0.0"
-                   izz="${2*mass*radius*radius/5}" />
-      </inertial>
+    <inertial>
+      <mass value="${mass}"/>
+      <origin xyz="0 0 0"/>
+      <inertia ixx="${2*mass*radius*radius/5}" ixy="0.0" ixz="0.0"
+               iyy="${2*mass*radius*radius/5}" iyz="0.0"
+               izz="${2*mass*radius*radius/5}"/>
+    </inertial>
   </xacro:macro>
   <xacro:macro name="sphere_geometry" params="radius">
@@ -21,11 +21,11 @@
   </xacro:macro>
   <xacro:macro name="cylinder_inertia" params="mass radius height">
-      <inertial>
-         <mass value="${mass}" />
-         <origin xyz="0 0 0" />
-         <inertia  ixx="${(3*radius*radius + height*height)*mass/12}" ixy="0.0" ixz="0.0"
-                   iyy="${(3*radius*radius + height*height)*mass/12}" iyz="0.0"
-                   izz="${radius*radius*mass/2}" />
-      </inertial>
+    <inertial>
+      <mass value="${mass}"/>
+      <origin xyz="0 0 0"/>
+      <inertia ixx="${(3*radius*radius + height*height)*mass/12}" ixy="0.0" ixz="0.0"
+               iyy="${(3*radius*radius + height*height)*mass/12}" iyz="0.0"
+               izz="${radius*radius*mass/2}"/>
+    </inertial>
   </xacro:macro>
   <xacro:macro name="cylinder_geometry" params="radius height">
@@ -40,11 +40,11 @@
   </xacro:macro>
   <xacro:macro name="box_inertia" params="mass width height depth">
-      <inertial>
-         <mass value="${mass}" />
-         <origin xyz="0 0 0" />
-         <inertia  ixx="${(depth*depth + height*height)*mass/12}" ixy="0.0" ixz="0.0"
-                   iyy="${(depth*depth + width*width)*mass/12}" iyz="0.0"
-                   izz="${(width*width + height*height)*mass/12}" />
-      </inertial>
+    <inertial>
+      <mass value="${mass}"/>
+      <origin xyz="0 0 0"/>
+      <inertia ixx="${(depth*depth + height*height)*mass/12}" ixy="0.0" ixz="0.0"
+               iyy="${(depth*depth + width*width)*mass/12}" iyz="0.0"
+               izz="${(width*width + height*height)*mass/12}"/>
+    </inertial>
   </xacro:macro>
   <xacro:macro name="box_geometry" params="width height depth">

File: moon_description/urdf/materials.urdf.xacro (robot description, xacro)
@@ -1,23 +1,23 @@
 <?xml version="1.0"?>
 <robot xmlns:xacro="http://www.ros.org/wiki/xacro">
-   <xacro:macro name="white_material">
-      <material name="white">
-        <color rgba="255 255 255 1"/>
-      </material>
-   </xacro:macro>
-   <xacro:macro name="black_material">
-      <material name="black">
-        <color rgba="0 0 0 1"/>
-      </material>
-   </xacro:macro>
-   <xacro:macro name="red_material">
-      <material name="red">
-        <color rgba="255 0 0 1"/>
-      </material>
-   </xacro:macro>
-   <xacro:macro name="green_material">
-      <material name="green">
-        <color rgba="0 255 0 1"/>
-      </material>
-   </xacro:macro>
+  <xacro:macro name="white_material">
+    <material name="white">
+      <color rgba="255 255 255 1"/>
+    </material>
+  </xacro:macro>
+  <xacro:macro name="black_material">
+    <material name="black">
+      <color rgba="0 0 0 1"/>
+    </material>
+  </xacro:macro>
+  <xacro:macro name="red_material">
+    <material name="red">
+      <color rgba="255 0 0 1"/>
+    </material>
+  </xacro:macro>
+  <xacro:macro name="green_material">
+    <material name="green">
+      <color rgba="0 255 0 1"/>
+    </material>
+  </xacro:macro>
 </robot>

File: moon_description/urdf/wheels.urdf.xacro (robot description, xacro)
@@ -1,61 +1,61 @@
 <?xml version="1.0"?>
 <robot xmlns:xacro="http://www.ros.org/wiki/xacro">
-    <xacro:macro name="caster_wheel" params="prefix radius x y z">
-        <link name="caster_${prefix}_wheel">
-            <visual>
-                <xacro:sphere_geometry radius="${radius}"/>
-                <xacro:black_material/>
-            </visual>
-            <xacro:sphere_collision radius="${radius}"/>
-            <xacro:sphere_inertia mass="0.05" radius="${radius}"/>
-        </link>
-        <joint name="caster_${prefix}_joint" type="fixed">
-            <parent link="base_link"/>
-            <child link="caster_${prefix}_wheel"/>
-            <origin rpy="0 0 0" xyz="${x} ${y} ${z}"/>
-        </joint>
-    </xacro:macro>
-    <xacro:macro name="transmission_wheel" params="prefix radius width holder_size wheels_distance direction">
-        <link name="${prefix}_wheel_holder">
-            <visual>
-                <xacro:box_geometry width="${holder_size}" height="${holder_size}" depth="${holder_size}"/>
-                <xacro:green_material/>
-            </visual>
-            <xacro:box_collision width="${holder_size}" height="${holder_size}" depth="${holder_size}"/>
-            <xacro:box_inertia mass="0.003" width="${holder_size}" height="${holder_size}" depth="${holder_size}"/>
-        </link>
-        <joint name="base_to_${prefix}_wheel_holder" type="fixed">
-            <parent link="base_link"/>
-            <child link="${prefix}_wheel_holder"/>
-            <origin xyz="${direction * (holder_size + wheels_distance)/2} 0 ${holder_size/2}" rpy="0 0 0" />
-            <axis xyz="0 0 1" />
-        </joint>
-        <link name="${prefix}_wheel">
-            <visual>
-                <xacro:cylinder_geometry radius="${radius}" height="${width}"/>
-                <xacro:black_material/>
-            </visual>
-            <xacro:cylinder_collision radius="${radius}" height="${width}"/>
-            <xacro:cylinder_inertia mass="0.03" radius="${radius}" height="${width}"/>
-            <dynamics damping="0.01" friction="100.0" />
-        </link>
-        <joint name="${prefix}_wheel_joint" type="continuous">
-            <parent link="${prefix}_wheel_holder"/>
-            <child link="${prefix}_wheel"/>
-            <origin xyz="${direction * (width + holder_size) / 2} 0 0" rpy="0 ${pi/2} 0" />
-            <axis xyz="0 0 1" />
-            <limit effort="100" velocity="100" />
-            <dynamics damping="0.01" friction="0.0" />
-        </joint>
-        <transmission name="${prefix}_wheel_transmission">
-            <type>transmission_interface/SimpleTransmission</type>
-            <joint name="${prefix}_wheel_joint">
-                <hardwareInterface>EffortJointInterface</hardwareInterface>
-            </joint>
-            <actuator name="${prefix}_wheel_motor">
-                <hardwareInterface>EffortJointInterface</hardwareInterface>
-                <mechanicalReduction>1</mechanicalReduction>
-            </actuator>
-        </transmission>
-    </xacro:macro>
+  <xacro:macro name="caster_wheel" params="prefix radius x y z">
+    <link name="caster_${prefix}_wheel">
+      <visual>
+        <xacro:sphere_geometry radius="${radius}"/>
+        <xacro:black_material/>
+      </visual>
+      <xacro:sphere_collision radius="${radius}"/>
+      <xacro:sphere_inertia mass="0.05" radius="${radius}"/>
+    </link>
+    <joint name="caster_${prefix}_joint" type="fixed">
+      <parent link="base_link"/>
+      <child link="caster_${prefix}_wheel"/>
+      <origin rpy="0 0 0" xyz="${x} ${y} ${z}"/>
+    </joint>
+  </xacro:macro>
+  <xacro:macro name="transmission_wheel" params="prefix radius width holder_size wheels_distance direction">
+    <link name="${prefix}_wheel_holder">
+      <visual>
+        <xacro:box_geometry width="${holder_size}" height="${holder_size}" depth="${holder_size}"/>
+        <xacro:green_material/>
+      </visual>
+      <xacro:box_collision width="${holder_size}" height="${holder_size}" depth="${holder_size}"/>
+      <xacro:box_inertia mass="0.003" width="${holder_size}" height="${holder_size}" depth="${holder_size}"/>
+    </link>
+    <joint name="base_to_${prefix}_wheel_holder" type="fixed">
+      <parent link="base_link"/>
+      <child link="${prefix}_wheel_holder"/>
+      <origin xyz="${direction * (holder_size + wheels_distance)/2} 0 ${holder_size/2}" rpy="0 0 0"/>
+      <axis xyz="0 0 1"/>
+    </joint>
+    <link name="${prefix}_wheel">
+      <visual>
+        <xacro:cylinder_geometry radius="${radius}" height="${width}"/>
+        <xacro:black_material/>
+      </visual>
+      <xacro:cylinder_collision radius="${radius}" height="${width}"/>
+      <xacro:cylinder_inertia mass="0.03" radius="${radius}" height="${width}"/>
+      <dynamics damping="0.01" friction="100.0"/>
+    </link>
+    <joint name="${prefix}_wheel_joint" type="continuous">
+      <parent link="${prefix}_wheel_holder"/>
+      <child link="${prefix}_wheel"/>
+      <origin xyz="${direction * (width + holder_size) / 2} 0 0" rpy="0 ${pi/2} 0"/>
+      <axis xyz="0 0 1"/>
+      <limit effort="100" velocity="100"/>
+      <dynamics damping="0.01" friction="0.0"/>
+    </joint>
+    <transmission name="${prefix}_wheel_transmission">
+      <type>transmission_interface/SimpleTransmission</type>
+      <joint name="${prefix}_wheel_joint">
+        <hardwareInterface>EffortJointInterface</hardwareInterface>
+      </joint>
+      <actuator name="${prefix}_wheel_motor">
+        <hardwareInterface>EffortJointInterface</hardwareInterface>
+        <mechanicalReduction>1</mechanicalReduction>
+      </actuator>
+    </transmission>
+  </xacro:macro>
 </robot>

Commit message: Added inertial tensor for combined shape of robot base

File: moon_description/robot/robot.urdf.xacro (robot description, xacro)
@@ -32,8 +32,14 @@
   <link name="base_link_inertia">
     <xacro:box_collision width="${base_width}" depth="${base_height}" height="${base_length}"/>
-    <xacro:box_inertia mass="3" width="${base_width}" depth="${base_height}" height="${base_length}"/>
+    <inertial>
+      <mass value="3.309"/>
+      <origin xyz="0.00331 0 0.03506"/>
+      <inertia ixx="2.547e-2" ixy="0.0" ixz="2.993e-6"
+               iyy="2.374e-2" iyz="0.0"
+               izz="4.650e-2"/>
+    </inertial>
   </link>
   <joint name="base_link_inertia_joint" type="fixed">
-    <origin xyz="${caster_radius} 0 ${caster_radius}" rpy="0 0 ${pi / 2}"/>
+    <origin xyz="0 0 0" rpy="0 0 0"/>
     <parent link="base_link"/>
     <child link="base_link_inertia"/>

Commit message: Fixed drift by adding mass to the wheels

File: moon_description/robot/robot.urdf.xacro (robot description, xacro)
@@ -31,15 +31,9 @@
   </link>
   <link name="base_link_inertia">
-    <xacro:box_collision width="${base_width}" depth="${base_height}" height="${base_length}"/>
-    <inertial>
-      <mass value="3.309"/>
-      <origin xyz="0.00331 0 0.03506"/>
-      <inertia ixx="2.547e-2" ixy="0.0" ixz="2.993e-6"
-               iyy="2.374e-2" iyz="0.0"
-               izz="4.650e-2"/>
-    </inertial>
+    <xacro:box_collision width="${base_length + 0.05}" depth="${base_height}" height="${base_width + 0.05}"/>
+    <xacro:box_inertia mass="3.0" width="${base_length}" depth="${base_height}" height="${base_width}"/>
   </link>
   <joint name="base_link_inertia_joint" type="fixed">
-    <origin xyz="0 0 0" rpy="0 0 0"/>
+    <origin xyz="0 0 ${base_height / 2}" rpy="0 0 0"/>
     <parent link="base_link"/>
     <child link="base_link_inertia"/>
@@ -49,8 +43,8 @@
   <xacro:transmission_wheel prefix="back_left" radius="${wheel_radius}" width="${wheel_width}"
                             holder_size="${wheel_holder_size}" direction="1.0" x="-0.0125" y="0.14"
-                            z="${wheel_radius - caster_radius}"/>
+                            z="${wheel_radius - caster_radius - 0.001}"/>
   <xacro:transmission_wheel prefix="back_right" radius="${wheel_radius}" width="${wheel_width}"
                             holder_size="${wheel_holder_size}" direction="-1.0" x="-0.0125" y="-0.14"
-                            z="${wheel_radius - caster_radius}"/>
+                            z="${wheel_radius - caster_radius - 0.001}"/>
   <xacro:caster_wheel prefix="back_left" radius="${caster_radius}" x="-0.1125" y="0.0725" z="0"/>
   <xacro:caster_wheel prefix="back_right" radius="${caster_radius}" x="-0.1125" y="-0.0725" z="0"/>

File: moon_description/urdf/wheels.urdf.xacro (robot description, xacro)
@@ -37,5 +37,5 @@
       </visual>
       <xacro:cylinder_collision radius="${radius}" height="${width}"/>
-      <xacro:cylinder_inertia mass="0.03" radius="${radius}" height="${width}"/>
+      <xacro:cylinder_inertia mass="1" radius="${radius}" height="${width}"/>
     </link>
     <joint name="${prefix}_wheel_joint" type="continuous">
