Commit message: Fixed simulation in Gazebo

File: moon_description/robot/moon.gazebo.xacro (robot description, xacro)
@@ -1,4 +1,4 @@
 <?xml version="1.0"?>
-<robot xmlns:xacro="http://www.ros.org/wiki/xacro" name="moon">
+<robot xmlns:xacro="http://ros.org/wiki/xacro" name="moon">
   <xacro:include filename="$(find moon_description)/robot/robot.urdf.xacro"/>
   <gazebo>
@@ -9,4 +9,6 @@
   </gazebo>
   <gazebo reference="base_link">
+    <mu1 value="0.0"/>
+    <mu2 value="0.0"/>
     <material>Gazebo/White</material>
   </gazebo>
@@ -14,3 +16,72 @@
     <turnGravityOff>false</turnGravityOff>
   </gazebo>
+  <gazebo reference="caster_front_left_wheel">
+    <mu1 value="0.0"/>
+    <mu2 value="0.0"/>
+    <material>Gazebo/Black</material>
+  </gazebo>
+  <gazebo reference="caster_front_right_wheel">
+    <mu1 value="0.0"/>
+    <mu2 value="0.0"/>
+    <material>Gazebo/Black</material>
+  </gazebo>
+  <gazebo reference="back_left_wheel_holder">
+    <mu1 value="0.0"/>
+    <mu2 value="0.0"/>
+    <kp value="10000000.0" />
+    <kd value="1.0" />
+    <material>Gazebo/White</material>
+  </gazebo>
+  <gazebo reference="back_left_wheel">
+    <mu1 value="1.0"/>
+    <mu2 value="1.0"/>
+    <kp value="10000000.0" />
+    <kd value="1.0" />
+    <material>Gazebo/Black</material>
+  </gazebo>
+  <gazebo reference="back_right_wheel_holder">
+    <mu1 value="0.0"/>
+    <mu2 value="0.0"/>
+    <kp value="10000000.0" />
+    <kd value="1.0" />
+    <material>Gazebo/White</material>
+  </gazebo>
+  <gazebo reference="back_right_wheel">
+    <mu1 value="1.0"/>
+    <mu2 value="1.0"/>
+    <kp value="10000000.0" />
+    <kd value="1.0" />
+    <material>Gazebo/Black</material>
+  </gazebo>
+  <gazebo reference="lidar">
+    <material>Gazebo/Green</material>
+    <sensor type="ray" name="hokuyo_sensor">
+      <pose>0 0 0.0124 0 0 0</pose>
+      <visualize>false</visualize>
+      <update_rate>40</update_rate>
+      <ray>
+        <scan>
+          <horizontal>
+            <samples>1081</samples>
+            <resolution>1</resolution>
+            <min_angle>-2.3561944902</min_angle>
+            <max_angle>2.3561944902</max_angle>
+          </horizontal>
+        </scan>
+        <range>
+          <min>0.1</min>
+          <max>10.0</max>
+          <resolution>0.01</resolution>
+        </range>
+        <noise>
+          <mean>0.0</mean>
+          <stddev>0.01</stddev>
+        </noise>
+      </ray>
+      <plugin name="gazebo_ros_hokuyo_controller" filename="libgazebo_ros_laser.so">
+        <topicName>/scan</topicName>
+        <frameName>laser</frameName>
+      </plugin>
+    </sensor>
+  </gazebo>
 </robot>

File: moon_description/robot/robot.urdf.xacro (robot description, xacro)
@@ -1,6 +1,4 @@
 <?xml version="1.0"?>
 <robot name="moon" xmlns:xacro="http://ros.org/wiki/xacro">
-  <!-- Global constants -->
-  <xacro:property name="pi" value="3.1415926535897931"/>
   <!-- Included files -->
   <xacro:include filename="$(find moon_description)/urdf/materials.urdf.xacro"/>
@@ -22,8 +20,7 @@
       <xacro:white_material/>
     </visual>
-    <xacro:box_inertia mass="0.0001" width="0.001" depth="0.001" height="0.001"/>
   </link>
   <joint name="base_footprint_joint" type="fixed">
-    <origin rpy="0 0 0" xyz="0 0 0.03"/>
+    <origin rpy="0 0 0" xyz="0 0 0.02"/>
     <parent link="base_footprint"/>
     <child link="base_link"/>

File: moon_description/urdf/wheels.urdf.xacro (robot description, xacro)
@@ -38,5 +38,4 @@
       <xacro:cylinder_collision radius="${radius}" height="${width}"/>
       <xacro:cylinder_inertia mass="0.03" radius="${radius}" height="${width}"/>
-      <dynamics damping="0.01" friction="100.0"/>
     </link>
     <joint name="${prefix}_wheel_joint" type="continuous">
@@ -45,6 +44,4 @@
       <origin xyz="${direction * (width + holder_size) / 2} 0 0" rpy="0 ${pi/2} 0"/>
       <axis xyz="0 0 1"/>
-      <limit effort="100" velocity="100"/>
-      <dynamics damping="0.01" friction="0.0"/>
     </joint>
     <transmission name="${prefix}_wheel_transmission">

Commit message: Saved experiments with odom fusion

File: moon_description/robot/moon.gazebo.xacro (robot description, xacro)
@@ -57,5 +57,5 @@
     <material>Gazebo/Green</material>
     <sensor type="ray" name="hokuyo_sensor">
-      <pose>0 0 0.0124 0 0 0</pose>
+      <pose>0 0 0 0 0 0</pose>
       <visualize>false</visualize>
       <update_rate>40</update_rate>
@@ -85,3 +85,17 @@
     </sensor>
   </gazebo>
+  <gazebo>
+    <plugin name="imu_controller" filename="libhector_gazebo_ros_imu.so">
+      <robotNamespace>/</robotNamespace>
+      <updateRate>50.0</updateRate>
+      <bodyName>imu_link</bodyName>
+      <topicName>imu/data</topicName>
+      <accelDrift>0.005 0.005 0.005</accelDrift>
+      <accelGaussianNoise>0.005 0.005 0.005</accelGaussianNoise>
+      <rateDrift>0.005 0.005 0.005 </rateDrift>
+      <rateGaussianNoise>0.005 0.005 0.005 </rateGaussianNoise>
+      <headingDrift>0.005</headingDrift>
+      <headingGaussianNoise>0.005</headingGaussianNoise>
+    </plugin>
+  </gazebo>
 </robot>

File: moon_description/robot/robot.urdf.xacro (robot description, xacro)
@@ -43,4 +43,15 @@
   <xacro:transmission_wheel prefix="back_right" radius="${wheel_radius}" width="${wheel_width}"
                             holder_size="${wheel_holder_size}" wheels_distance="0.05" direction="-1.0"/>
+  <joint name="imu_link_joint" type="fixed">
+    <origin rpy="0 0 0" xyz="0 0 -0.01"/>
+    <parent link="base_link"/>
+    <child link="imu_link"/>
+  </joint>
+  <link name="imu_link">
+    <visual>
+      <xacro:box_geometry width="0.001" depth="0.001" height="0.001"/>
+      <xacro:white_material/>
+    </visual>
+  </link>
   <link name="lidar">
     <visual>
@@ -50,5 +61,4 @@
     <xacro:cylinder_collision radius="${lidar_radius}" height="${lidar_height}"/>
     <xacro:cylinder_inertia mass="0.1" radius="${lidar_radius}" height="${lidar_height}"/>
-    <dynamics damping="0.01" friction="100.0"/>
   </link>
   <joint name="lidar_joint" type="fixed">

Commit message: Fixed inertia issues and added rotated base_link.

File: moon_description/robot/moon.gazebo.xacro (robot description, xacro)
@@ -29,6 +29,6 @@
     <mu1 value="0.0"/>
     <mu2 value="0.0"/>
-    <kp value="10000000.0" />
-    <kd value="1.0" />
+    <kp value="10000000.0"/>
+    <kd value="1.0"/>
     <material>Gazebo/White</material>
   </gazebo>
@@ -36,6 +36,6 @@
     <mu1 value="1.0"/>
     <mu2 value="1.0"/>
-    <kp value="10000000.0" />
-    <kd value="1.0" />
+    <kp value="10000000.0"/>
+    <kd value="1.0"/>
     <material>Gazebo/Black</material>
   </gazebo>
@@ -43,6 +43,6 @@
     <mu1 value="0.0"/>
     <mu2 value="0.0"/>
-    <kp value="10000000.0" />
-    <kd value="1.0" />
+    <kp value="10000000.0"/>
+    <kd value="1.0"/>
     <material>Gazebo/White</material>
   </gazebo>
@@ -50,6 +50,6 @@
     <mu1 value="1.0"/>
     <mu2 value="1.0"/>
-    <kp value="10000000.0" />
-    <kd value="1.0" />
+    <kp value="10000000.0"/>
+    <kd value="1.0"/>
     <material>Gazebo/Black</material>
   </gazebo>
@@ -57,5 +57,5 @@
     <material>Gazebo/Green</material>
     <sensor type="ray" name="hokuyo_sensor">
-      <pose>0 0 0.0124 0 0 0</pose>
+      <pose>0 0 0 0 0 0</pose>
       <visualize>false</visualize>
       <update_rate>40</update_rate>

File: moon_description/robot/robot.urdf.xacro (robot description, xacro)
@@ -15,10 +15,5 @@
   <xacro:property name="lidar_height" value="0.02"/>
   <xacro:property name="lidar_radius" value="0.04"/>
-  <link name="base_footprint">
-    <visual>
-      <xacro:box_geometry width="0.001" depth="0.001" height="0.001"/>
-      <xacro:white_material/>
-    </visual>
-  </link>
+  <link name="base_footprint"/>
   <joint name="base_footprint_joint" type="fixed">
     <origin rpy="0 0 0" xyz="0 0 0.02"/>
@@ -34,9 +29,16 @@
       <xacro:white_material/>
     </visual>
+  </link>
+  <link name="base_link_inertia">
     <xacro:box_collision width="${base_width}" depth="${base_height}" height="${base_length}"/>
     <xacro:box_inertia mass="3" width="${base_width}" depth="${base_height}" height="${base_length}"/>
   </link>
-  <xacro:caster_wheel prefix="front_left" radius="${caster_radius}" x="0.05" y="-0.1" z="0"/>
-  <xacro:caster_wheel prefix="front_right" radius="${caster_radius}" x="-0.05" y="-0.1" z="0"/>
+  <joint name="base_link_inertia_joint" type="fixed">
+    <origin xyz="${caster_radius} 0 ${caster_radius}" rpy="0 0 ${pi / 2}"/>
+    <parent link="base_link"/>
+    <child link="base_link_inertia"/>
+  </joint>
+  <xacro:caster_wheel prefix="front_left" radius="${caster_radius}" x="0.1" y="0.05" z="0"/>
+  <xacro:caster_wheel prefix="front_right" radius="${caster_radius}" x="0.1" y="-0.05" z="0"/>
   <xacro:transmission_wheel prefix="back_left" radius="${wheel_radius}" width="${wheel_width}"
                             holder_size="${wheel_holder_size}" wheels_distance="0.05" direction="1.0"/>
@@ -53,5 +55,5 @@
   </link>
   <joint name="lidar_joint" type="fixed">
-    <origin rpy="0 0 0" xyz="0 0.04 ${base_height + lidar_height/2}"/>
+    <origin rpy="0 0 0" xyz="-0.04 0 ${base_height + lidar_height/2}"/>
     <parent link="base_link"/>
     <child link="lidar"/>

File: moon_description/urdf/common.urdf.xacro (robot description, xacro)
@@ -10,7 +10,27 @@
     </inertial>
   </xacro:macro>
+  <xacro:macro name="sphere_inertia_gazebo" params="mass radius">
+    <inertial>
+      <mass>${mass}</mass>
+      <inertia>
+        <ixx>${2*mass*radius*radius/5}</ixx>
+        <ixy>0</ixy>
+        <iyy>${2*mass*radius*radius/5}</iyy>
+        <ixz>0</ixz>
+        <iyz>0</iyz>
+        <izz>${2*mass*radius*radius/5}</izz>
+      </inertia>
+    </inertial>
+  </xacro:macro>
   <xacro:macro name="sphere_geometry" params="radius">
     <geometry>
       <sphere radius="${radius}"/>
+    </geometry>
+  </xacro:macro>
+  <xacro:macro name="sphere_geometry_gazebo" params="radius">
+    <geometry>
+      <sphere>
+        <radius>${radius}</radius>
+      </sphere>
     </geometry>
   </xacro:macro>

File: moon_description/urdf/wheels.urdf.xacro (robot description, xacro)
@@ -28,5 +28,5 @@
       <parent link="base_link"/>
       <child link="${prefix}_wheel_holder"/>
-      <origin xyz="${direction * (holder_size + wheels_distance)/2} 0 ${holder_size/2}" rpy="0 0 0"/>
+      <origin xyz="0 ${direction * (holder_size + wheels_distance)/2} ${holder_size/2}" rpy="0 0 ${pi / 2}"/>
       <axis xyz="0 0 1"/>
     </joint>

Commit message: Development commit. Realistic robot. Issues in simulation with base_footprint.

File: moon_description/robot/moon.gazebo.xacro (robot description, xacro)
@@ -38,4 +38,14 @@
     <kp value="10000000.0"/>
     <kd value="1.0"/>
+    <material>Gazebo/Black</material>
+  </gazebo>
+  <gazebo reference="caster_back_left_wheel">
+    <mu1 value="0.0"/>
+    <mu2 value="0.0"/>
+    <material>Gazebo/Black</material>
+  </gazebo>
+  <gazebo reference="caster_back_right_wheel">
+    <mu1 value="0.0"/>
+    <mu2 value="0.0"/>
     <material>Gazebo/Black</material>
   </gazebo>

File: moon_description/robot/robot.urdf.xacro (robot description, xacro)
@@ -6,16 +6,16 @@
   <xacro:include filename="$(find moon_description)/urdf/wheels.urdf.xacro"/>
   <!-- Robot properties -->
-  <xacro:property name="base_width" value="0.2"/>
-  <xacro:property name="base_length" value="0.26"/>
-  <xacro:property name="base_height" value="0.06"/>
-  <xacro:property name="caster_radius" value="0.03"/>
-  <xacro:property name="wheel_width" value="0.02"/>
-  <xacro:property name="wheel_radius" value="0.035"/>
+  <xacro:property name="base_width" value="0.325"/>
+  <xacro:property name="base_length" value="0.3"/>
+  <xacro:property name="base_height" value="0.07"/>
+  <xacro:property name="caster_radius" value="0.008"/>
+  <xacro:property name="wheel_width" value="0.015"/>
+  <xacro:property name="wheel_radius" value="0.0375"/>
   <xacro:property name="wheel_holder_size" value="0.01"/>
   <xacro:property name="lidar_height" value="0.02"/>
-  <xacro:property name="lidar_radius" value="0.04"/>
+  <xacro:property name="lidar_radius" value="0.045"/>
   <link name="base_footprint"/>
   <joint name="base_footprint_joint" type="fixed">
-    <origin rpy="0 0 0" xyz="0 0 0.02"/>
+    <origin rpy="0 0 0" xyz="0 0 0.001"/>
     <parent link="base_footprint"/>
     <child link="base_link"/>
@@ -39,10 +39,14 @@
     <child link="base_link_inertia"/>
   </joint>
-  <xacro:caster_wheel prefix="front_left" radius="${caster_radius}" x="0.1" y="0.05" z="0"/>
-  <xacro:caster_wheel prefix="front_right" radius="${caster_radius}" x="0.1" y="-0.05" z="0"/>
+  <xacro:caster_wheel prefix="front_left" radius="${caster_radius}" x="0.0675" y="0.0725" z="0"/>
+  <xacro:caster_wheel prefix="front_right" radius="${caster_radius}" x="0.0675" y="-0.0725" z="0"/>
   <xacro:transmission_wheel prefix="back_left" radius="${wheel_radius}" width="${wheel_width}"
-                            holder_size="${wheel_holder_size}" wheels_distance="0.05" direction="1.0"/>
+                            holder_size="${wheel_holder_size}" direction="1.0" x="-0.0125" y="0.14"
+                            z="${wheel_radius - caster_radius}"/>
   <xacro:transmission_wheel prefix="back_right" radius="${wheel_radius}" width="${wheel_width}"
-                            holder_size="${wheel_holder_size}" wheels_distance="0.05" direction="-1.0"/>
+                            holder_size="${wheel_holder_size}" direction="-1.0" x="-0.0125" y="-0.14"
+                            z="${wheel_radius - caster_radius}"/>
+  <xacro:caster_wheel prefix="back_left" radius="${caster_radius}" x="-0.1125" y="0.0725" z="0"/>
+  <xacro:caster_wheel prefix="back_right" radius="${caster_radius}" x="-0.1125" y="-0.0725" z="0"/>
   <link name="lidar">
     <visual>

File: moon_description/urdf/wheels.urdf.xacro (robot description, xacro)
@@ -16,5 +16,5 @@
     </joint>
   </xacro:macro>
-  <xacro:macro name="transmission_wheel" params="prefix radius width holder_size wheels_distance direction">
+  <xacro:macro name="transmission_wheel" params="prefix radius width holder_size direction x y z">
     <link name="${prefix}_wheel_holder">
       <visual>
@@ -28,5 +28,5 @@
       <parent link="base_link"/>
       <child link="${prefix}_wheel_holder"/>
-      <origin xyz="0 ${direction * (holder_size + wheels_distance)/2} ${holder_size/2}" rpy="0 0 ${pi / 2}"/>
+      <origin xyz="${x} ${y} ${z}" rpy="0 0 ${pi / 2}"/>
       <axis xyz="0 0 1"/>
     </joint>
@@ -42,5 +42,5 @@
       <parent link="${prefix}_wheel_holder"/>
       <child link="${prefix}_wheel"/>
-      <origin xyz="${direction * (width + holder_size) / 2} 0 0" rpy="0 ${pi/2} 0"/>
+      <origin xyz="${-direction * (width + holder_size) / 2} 0 0" rpy="0 ${pi/2} 0"/>
       <axis xyz="0 0 1"/>
     </joint>

Commit message: Spread weight on the forward caster wheels. Fixed materials codding issue. Robot is navigating with small errors. Probably need more calibration of control.

File: moon_description/robot/moon.gazebo.xacro (robot description, xacro)
@@ -11,5 +11,5 @@
     <mu1 value="0.0"/>
     <mu2 value="0.0"/>
-    <material>Gazebo/White</material>
+    <material>Gazebo/Gold</material>
   </gazebo>
   <gazebo reference="base_footprint">

File: moon_description/robot/robot.urdf.xacro (robot description, xacro)
@@ -27,5 +27,5 @@
         <mesh filename="package://moon_description/meshes/moon_base.stl"/>
       </geometry>
-      <xacro:white_material/>
+      <xacro:navajo_white_material/>
     </visual>
   </link>
@@ -39,6 +39,6 @@
     <child link="base_link_inertia"/>
   </joint>
-  <xacro:caster_wheel prefix="front_left" radius="${caster_radius}" x="0.0675" y="0.0725" z="0"/>
-  <xacro:caster_wheel prefix="front_right" radius="${caster_radius}" x="0.0675" y="-0.0725" z="0"/>
+  <xacro:caster_wheel prefix="front_left" radius="${caster_radius}" x="0.12" y="0.12" z="0"/>
+  <xacro:caster_wheel prefix="front_right" radius="${caster_radius}" x="0.12" y="-0.12" z="0"/>
   <xacro:transmission_wheel prefix="back_left" radius="${wheel_radius}" width="${wheel_width}"
                             holder_size="${wheel_holder_size}" direction="1.0" x="-0.0125" y="0.14"
@@ -47,6 +47,6 @@
                             holder_size="${wheel_holder_size}" direction="-1.0" x="-0.0125" y="-0.14"
                             z="${wheel_radius - caster_radius}"/>
-  <xacro:caster_wheel prefix="back_left" radius="${caster_radius}" x="-0.1125" y="0.0725" z="0"/>
-  <xacro:caster_wheel prefix="back_right" radius="${caster_radius}" x="-0.1125" y="-0.0725" z="0"/>
+  <xacro:caster_wheel prefix="back_left" radius="${caster_radius - 0.0001}" x="-0.1125" y="0.0725" z="0"/>
+  <xacro:caster_wheel prefix="back_right" radius="${caster_radius - 0.0001}" x="-0.1125" y="-0.0725" z="0"/>
   <link name="lidar">
     <visual>

File: moon_description/urdf/materials.urdf.xacro (robot description, xacro)
@@ -3,20 +3,25 @@
   <xacro:macro name="white_material">
     <material name="white">
-      <color rgba="255 255 255 1"/>
+      <color rgba="1.0 1.0 1.0 1.0"/>
     </material>
   </xacro:macro>
   <xacro:macro name="black_material">
     <material name="black">
-      <color rgba="0 0 0 1"/>
+      <color rgba="0.0 0.0 0.0 1.0"/>
+    </material>
+  </xacro:macro>
+  <xacro:macro name="navajo_white_material">
+    <material name="navajo_white">
+      <color rgba="1.0 0.87 0.68 1.0"/>
     </material>
   </xacro:macro>
   <xacro:macro name="red_material">
     <material name="red">
-      <color rgba="255 0 0 1"/>
+      <color rgba="1.0 0.0 0.0 1.0"/>
     </material>
   </xacro:macro>
   <xacro:macro name="green_material">
     <material name="green">
-      <color rgba="0 255 0 1"/>
+      <color rgba="0.0 1.0 0.0 1.0"/>
     </material>
   </xacro:macro>
